File: Hardware/PCB/attenuverters/attenuverters.sch (KiCad schematic (older format))
At the start: 62 parts, among them J1 AudioJack2, J10 Conn_01x16, J11 Conn_01x16, J12 3_pin_Molex_header, J13 3_pin_Molex_connector, J2 AudioJack2, J3 AudioJack2, J4 AudioJack2, J5 AudioJack2_SwitchT, J6 AudioJack2_SwitchT, J7 AudioJack2_SwitchT, J8 Synth_power_2x5, J9 AudioJack2, SW1 SW_SPDT, U1 TL072, U2 TL072, U3 TL071, U4 LM4040DIZ-10.0

Commit message: k not K; BOM
Parts:
- R19, R24: value 1K -> 1k
Changed lines of the file:
@@
 P 4800 6650
 F 0 "R19" V 4593 6650 50  0000 C CNN
-F 1 "1K" V 4684 6650 50  0000 C CNN
+F 1 "1k" V 4684 6650 50  0000 C CNN
 F 2 "ao_tht:R_Axial_DIN0207_L6.3mm_D2.5mm_P10.16mm_Horizontal" V 4730 6650 50  0001 C CNN
 F 3 "" H 4800 6650 50  0001 C CNN
@@
 P 4800 7400
 F 0 "R24" V 4593 7400 50  0000 C CNN
-F 1 "1K" V 4684 7400 50  0000 C CNN
+F 1 "1k" V 4684 7400 50  0000 C CNN
 F 2 "ao_tht:R_Axial_DIN0207_L6.3mm_D2.5mm_P10.16mm_Horizontal" V 4730 7400 50  0001 C CNN
 F 3 "" H 4800 7400 50  0001 C CNN
@@
 $EndComp
 $Comp
-L attenuverters:+10V_P #PWR?
+L attenuverters:+10V_P #PWR0109
 U 1 1 616F61AE
 P 5950 4100
-F 0 "#PWR?" H 5950 3950 50  0001 C CNN
+F 0 "#PWR0109" H 5950 3950 50  0001 C CNN
 F 1 "+10V_P" H 5965 4273 50  0000 C CNN
 F 2 "" H 5950 4100 50  0001 C CNN

Commit message: Revised PCB
Parts:
- removed R25: 100k, ao_tht:R_Axial_DIN0207_L6.3mm_D2.5mm_P10.16mm_Horizontal, symbol ao_symbols:R
- C1, C2: symbol Device:CP -> ao_symbols:CP
- C3, C4, C5, C6, C7, C8: symbol Device:C -> ao_symbols:C
- D1, D2: symbol Device:D_Schottky -> ao_symbols:1N5817
- R1, R2, R3: value 10k -> 9.1k
- R20, R21, R22: value 100k -> 1k
Connections:
- wire segments 174 -> 173
Changed lines of the file:
@@
 $EndDescr
 $Comp
-L Device:D_Schottky D1
+L ao_symbols:1N5817 D1
 U 1 1 5F73FA24
 P 8100 1250
@@
 $EndComp
 $Comp
-L Device:CP C1
+L ao_symbols:CP C1
 U 1 1 5F73FA30
 P 6550 2500
@@
 Connection ~ 7400 1250
 $Comp
-L Device:D_Schottky D2
+L ao_symbols:1N5817 D2
 U 1 1 6074E3B2
 P 8100 1650
@@
 $EndComp
 $Comp
-L Device:CP C2
+L ao_symbols:CP C2
 U 1 1 6074E7B5
 P 6550 2800
@@
 Connection ~ 6550 2650
 $Comp
-L Device:C C4
+L ao_symbols:C C4
 U 1 1 6074ED42
 P 7200 2800
@@
 P 2850 1900
 F 0 "R20" V 2643 1900 50  0000 C CNN
-F 1 "100k" V 2734 1900 50  0000 C CNN
+F 1 "1k" V 2734 1900 50  0000 C CNN
 F 2 "ao_tht:R_Axial_DIN0207_L6.3mm_D2.5mm_P10.16mm_Horizontal" V 2780 1900 50  0001 C CNN
 F 3 "" H 2850 1900 50  0001 C CNN
@@
 P 2850 3400
 F 0 "R21" V 2643 3400 50  0000 C CNN
-F 1 "100k" V 2734 3400 50  0000 C CNN
+F 1 "1k" V 2734 3400 50  0000 C CNN
 F 2 "ao_tht:R_Axial_DIN0207_L6.3mm_D2.5mm_P10.16mm_Horizontal" V 2780 3400 50  0001 C CNN
 F 3 "" H 2850 3400 50  0001 C CNN
@@
 P 2850 4900
 F 0 "R22" V 2643 4900 50  0000 C CNN
-F 1 "100k" V 2734 4900 50  0000 C CNN
+F 1 "1k" V 2734 4900 50  0000 C CNN
 F 2 "ao_tht:R_Axial_DIN0207_L6.3mm_D2.5mm_P10.16mm_Horizontal" V 2780 4900 50  0001 C CNN
 F 3 "" H 2850 4900 50  0001 C CNN
@@
 P 1950 6450
 F 0 "R1" V 1850 6350 50  0000 C CNN
-F 1 "10k" V 1850 6550 50  0000 C CNN
+F 1 "9.1k" V 1850 6550 50  0000 C CNN
 F 2 "ao_tht:R_Axial_DIN0207_L6.3mm_D2.5mm_P10.16mm_Horizontal" V 1880 6450 50  0001 C CNN
 F 3 "" H 1950 6450 50  0001 C CNN
@@
 P 1950 6650
 F 0 "R2" V 1850 6550 50  0000 C CNN
-F 1 "10k" V 1850 6750 50  0000 C CNN
+F 1 "9.1k" V 1850 6750 50  0000 C CNN
 F 2 "ao_tht:R_Axial_DIN0207_L6.3mm_D2.5mm_P10.16mm_Horizontal" V 1880 6650 50  0001 C CNN
 F 3 "" H 1950 6650 50  0001 C CNN
@@
 P 1950 6850
 F 0 "R3" V 1850 6750 50  0000 C CNN
-F 1 "10k" V 1850 6950 50  0000 C CNN
+F 1 "9.1k" V 1850 6950 50  0000 C CNN
 F 2 "ao_tht:R_Axial_DIN0207_L6.3mm_D2.5mm_P10.16mm_Horizontal" V 1880 6850 50  0001 C CNN
 F 3 "" H 1950 6850 50  0001 C CNN
@@
 Connection ~ 7200 2950
 $Comp
-L Device:C C7
+L ao_symbols:C C7
 U 1 1 61743108
 P 8200 2500
@@
 $EndComp
 $Comp
-L Device:C C8
+L ao_symbols:C C8
 U 1 1 61743123
 P 8200 2800
@@
 Connection ~ 9350 2650
 $Comp
-L Device:C C6
+L ao_symbols:C C6
 U 1 1 6174B8E9
 P 9350 2800
@@
 $EndComp
 $Comp
-L Device:C C5
+L ao_symbols:C C5
 U 1 1 6174B8CE
 P 9350 2500
@@
 Wire Wire Line
 	6950 5700 6950 5600
-$Comp
-L ao_symbols:R R25
-U 1 1 61B95A69
-P 6200 4200
-F 0 "R25" V 5993 4200 50  0000 C CNN
-F 1 "100k" V 6084 4200 50  0000 C CNN
-F 2 "ao_tht:R_Axial_DIN0207_L6.3mm_D2.5mm_P10.16mm_Horizontal" V 6130 4200 50  0001 C CNN
-F 3 "" H 6200 4200 50  0001 C CNN
-F 4 "Tayda" H 6200 4200 50  0001 C CNN "Vendor"
-	1    6200 4200
-	0    1    1    0
-$EndComp
-Wire Wire Line
-	5950 4200 6050 4200
 Text GLabel 7200 6250 2    50   Output ~ 0
 NONINV3_P
@@
 NONINV3_P
 $Comp
-L Device:C C3
+L ao_symbols:C C3
 U 1 1 5F73FA42
 P 7200 2500
@@
 U 1 1 61CDDFFB
 P 6700 3950
-F 0 "J12" V 6664 3762 50  0000 R CNN
-F 1 "3_pin_Molex_header" V 6573 3762 50  0000 R CNN
+F 0 "J12" V 6750 4300 50  0000 R CNN
+F 1 "3_pin_Molex_header" V 6650 4900 50  0000 R CNN
 F 2 "ao_tht:Molex_KK-254_AE-6410-03A_1x03_P2.54mm_Vertical" H 6700 3950 50  0001 C CNN
 F 3 "" H 6700 3950 50  0001 C CNN
@@
 F 5 "A-805" H 6700 3950 50  0001 C CNN "SKU"
 	1    6700 3950
-	0    -1   -1   0
+	0    1    -1   0
 $EndComp
 Wire Wire Line
 	6600 4200 6600 4150
-Wire Wire Line
-	6350 4200 6600 4200
 Wire Wire Line
 	6700 4150 6700 4300
@@
 	1    0    0    -1
 $EndComp
+Wire Wire Line
+	5950 4200 6600 4200
 $EndSCHEMATC

Commit message: 2x072->074, correct wrong power connections
Parts:
- removed C5, C6: 100nF, ao_tht:C_Disc_D3.0mm_W1.6mm_P2.50mm, symbol ao_symbols:C
- removed unit 3 of U1
- U1: renamed from U2; value TL072 -> TL074; footprint ao_tht:DIP-8_W7.62mm_Socket_LongPads -> ao_tht:DIP-14_W7.62mm_Socket_LongPads; symbol ao_symbols:TL072 -> ao_symbols:TL074; SKU A-037 -> A-1138
- U1: value TL072 -> TL074; footprint ao_tht:DIP-8_W7.62mm_Socket_LongPads -> ao_tht:DIP-14_W7.62mm_Socket_LongPads; symbol ao_symbols:TL072 -> ao_symbols:TL074; SKU A-037 -> A-1138
- U1: renamed from U2; value TL072 -> TL074; footprint ao_tht:DIP-8_W7.62mm_Socket_LongPads -> ao_tht:DIP-14_W7.62mm_Socket_LongPads; symbol ao_symbols:TL072 -> ao_symbols:TL074
- renumbered C7 to C5, C8 to C6, J11 to J1, J6 to J10, J7 to J11, J4 to J12, J9 to J13, J10 to J2, J1 to J3, J2 to J4, J3 to J5, J12 to J6, J8 to J7, J13 to J8, J5 to J9, R6 to R1, R1 to R10, R2 to R11, R3 to R12, R16 to R13, R17 to R14, R18 to R15, R20 to R16, R21 to R17, R22 to R18, R4 to R19, R7 to R2, R5 to R20, R15 to R21, R19 to R22, R24 to R23, R23 to R24, R8 to R3, R9 to R4, R10 to R5, R11 to R6, R12 to R7, R13 to R8, R14 to R9, U3 to U2, U4 to U3
Connections:
- net labels added: 10V_REF, 10V_REF_P
- net labels removed: +10V, +10V_P
- wire segments 173 -> 167

Commit message: Test points
Parts:
- added TP1: GND, ao_tht:TestPoint_THTPad_1.5x1.5mm_Drill0.7mm, symbol ao_symbols:TestPoint
- added TP2: +12V, ao_tht:TestPoint_THTPad_D1.5mm_Drill0.7mm, symbol ao_symbols:TestPoint
- added TP3: -12V, ao_tht:TestPoint_THTPad_D1.5mm_Drill0.7mm, symbol ao_symbols:TestPoint
- added TP4: GND, ao_tht:TestPoint_THTPad_1.5x1.5mm_Drill0.7mm, symbol Connector:TestPoint
Connections:
- net +12V: now also TP2.1
- net -12V: now also TP3.1
- net GND: now also TP1.1
- net GND1: now also TP4.1
Changed lines of the file:
@@
 	1    0    0    1
 $EndComp
+$Comp
+L ao_symbols:TestPoint TP1
+U 1 1 61971C6A
+P 9750 2350
+F 0 "TP1" H 9808 2468 50  0000 L CNN
+F 1 "GND" H 9808 2377 50  0000 L CNN
+F 2 "ao_tht:TestPoint_THTPad_1.5x1.5mm_Drill0.7mm" H 9950 2350 50  0001 C CNN
+F 3 "~" H 9950 2350 50  0001 C CNN
+	1    9750 2350
+	1    0    0    -1
+$EndComp
+$Comp
+L ao_symbols:TestPoint TP2
+U 1 1 61972020
+P 9750 2650
+F 0 "TP2" H 9808 2768 50  0000 L CNN
+F 1 "+12V" H 9808 2677 50  0000 L CNN
+F 2 "ao_tht:TestPoint_THTPad_D1.5mm_Drill0.7mm" H 9950 2650 50  0001 C CNN
+F 3 "~" H 9950 2650 50  0001 C CNN
+	1    9750 2650
+	1    0    0    -1
+$EndComp
+$Comp
+L ao_symbols:TestPoint TP3
+U 1 1 6197240E
+P 9750 2950
+F 0 "TP3" H 9808 3068 50  0000 L CNN
+F 1 "-12V" H 9808 2977 50  0000 L CNN
+F 2 "ao_tht:TestPoint_THTPad_D1.5mm_Drill0.7mm" H 9950 2950 50  0001 C CNN
+F 3 "~" H 9950 2950 50  0001 C CNN
+	1    9750 2950
+	1    0    0    -1
+$EndComp
+$Comp
+L power:+12V #PWR037
+U 1 1 6197281C
+P 9750 2650
+F 0 "#PWR037" H 9750 2500 50  0001 C CNN
+F 1 "+12V" H 9765 2823 50  0000 C CNN
+F 2 "" H 9750 2650 50  0001 C CNN
+F 3 "" H 9750 2650 50  0001 C CNN
+	1    9750 2650
+	0    -1   -1   0
+$EndComp
+$Comp
+L power:-12V #PWR038
+U 1 1 61972D00
+P 9750 2950
+F 0 "#PWR038" H 9750 3050 50  0001 C CNN
+F 1 "-12V" H 9765 3123 50  0000 C CNN
+F 2 "" H 9750 2950 50  0001 C CNN
+F 3 "" H 9750 2950 50  0001 C CNN
+	1    9750 2950
+	0    -1   -1   0
+$EndComp
+$Comp
+L power:GND #PWR036
+U 1 1 61973167
+P 9750 2350
+F 0 "#PWR036" H 9750 2100 50  0001 C CNN
+F 1 "GND" H 9755 2177 50  0000 C CNN
+F 2 "" H 9750 2350 50  0001 C CNN
+F 3 "" H 9750 2350 50  0001 C CNN
+	1    9750 2350
+	0    1    1    0
+$EndComp
+$Comp
+L Connector:TestPoint TP4
+U 1 1 61983DFB
+P 9750 3950
+F 0 "TP4" H 9808 4068 50  0000 L CNN
+F 1 "GND" H 9808 3977 50  0000 L CNN
+F 2 "ao_tht:TestPoint_THTPad_1.5x1.5mm_Drill0.7mm" H 9950 3950 50  0001 C CNN
+F 3 "~" H 9950 3950 50  0001 C CNN
+	1    9750 3950
+	1    0    0    -1
+$EndComp
+$Comp
+L power:GND1 #PWR039
+U 1 1 6198B494
+P 9750 3950
+F 0 "#PWR039" H 9750 3700 50  0001 C CNN
+F 1 "GND1" H 9755 3777 50  0000 C CNN
+F 2 "" H 9750 3950 50  0001 C CNN
+F 3 "" H 9750 3950 50  0001 C CNN
+	1    9750 3950
+	0    1    1    0
+$EndComp
 $EndSCHEMATC
