File: Hardware/PCB/attenuverters/attenuverters.kicad_pcb (KiCad board)
At the start: 2 copper layers, 158 x 165 mm, 62 parts, among them J1 AudioJack2, J10 Conn_01x16, J11 Conn_01x16, J12 3_pin_Molex_header, J13 3_pin_Molex_connector, J2 AudioJack2, J3 AudioJack2, J4 AudioJack2, J5 AudioJack2_SwitchT, J6 AudioJack2_SwitchT, J7 AudioJack2_SwitchT, J8 Synth_power_2x5, J9 AudioJack2, SW1 SW_SPDT, U1 TL072, U2 TL072, U3 TL071, U4 LM4040DIZ-10.0

Commit message: Revised PCB
Parts:
- removed R25: 100k, ao_tht:R_Axial_DIN0207_L6.3mm_D2.5mm_P10.16mm_Horizontal
- R1, R2, R3: value 10k -> 9.1k
- R19, R24: value 1K -> 1k
- R20, R21, R22: value 100k -> 1k
- moved GRAF2 169.8 mm to (213.4, 58.0), turned to 270 degrees
- moved R9 68.4 mm to (190.5, 131.7), turned to 180 degrees
- moved R7 67.2 mm to (208.3, 132.9), turned to 0 degrees
- moved R14 64.7 mm to (208.3, 66.9), turned to 0 degrees
- moved C8 64.6 mm to (199.4, 67.1), turned to 180 degrees
- moved C3 61.4 mm to (203.2, 129.1), turned to 180 degrees
- moved R8 58.6 mm to (190.5, 126.6), turned to 180 degrees
- moved R22 57.6 mm to (180.3, 83.4), turned to 0 degrees
- moved R6 57.4 mm to (208.3, 127.9), turned to 0 degrees
- moved U3 56.4 mm to (203.2, 70.7), turned to 180 degrees
- moved R10 55.0 mm to (208.3, 72.0), turned to 0 degrees
- moved R13 49.1 mm to (190.5, 121.5), turned to 180 degrees
- moved R12 47.9 mm to (208.3, 122.8), turned to 0 degrees
- moved R18 47.7 mm to (190.5, 77.2), turned to 180 degrees
- moved R24 46.5 mm to (218.4, 87.2), turned to 180 degrees
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Connections:
- J12 pad 1: Net-(J12-Pad1) -> Net-(J1-PadT)
- J12 pad 3: Net-(J1-PadT) -> +10V_P
Routing:
- net INV2: track 94.6 -> 27.1 mm
- net INV3: track 21.4 -> 85.0 mm
- net NONINV2: track 91.6 -> 30.0 mm, vias 1 -> 0
- net INV1: track 94.6 -> 38.5 mm
- net NONINV3: track 38.5 -> 87.1 mm
- net OUT2: track 79.2 -> 42.4 mm
- net OUT3: track 46.6 -> 78.5 mm
- net OUT~SUM~: track 26.4 -> 55.4 mm
- net NONINV1: track 99.2 -> 72.1 mm
- net OUT1: track 69.6 -> 43.1 mm
- net Net-(J12-Pad1): track 18.8 -> 0.00 mm
- net Net-(J1-PadT): track 21.6 -> 38.8 mm
- net +10V: track 100.0 -> 83.1 mm
- net /-12_IN: track 25.4 -> 10.2 mm
- net SUM1: track 65.2 -> 51.9 mm
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Other:
- outline, holes or cut-outs redrawn

Commit message: 2x072->074, correct wrong power connections
Parts:
- removed the C5 at (203.2, 105.0)
- removed the C6 at (198.1, 89.8)
- removed the U1 at (203.2, 93.6)
- U1: renamed from U2; value TL072 -> TL074; footprint ao_tht:DIP-8_W7.62mm_Socket_LongPads -> ao_tht:DIP-14_W7.62mm_Socket_LongPads
- moved RV1 70.1 mm to (73.0, 100.0), turned to 90 degrees
- moved RV2 70.1 mm to (98.0, 100.0), turned to 90 degrees
- moved RV3 70.1 mm to (123.0, 100.0), turned to 90 degrees
- moved C3 33.0 mm to (203.2, 96.1)
- moved R18 28.4 mm to (208.4, 79.1)
- moved R15 28.2 mm to (218.6, 74.5)
- moved R5 28.1 mm to (180.3, 74.5)
- moved R9 25.1 mm to (190.5, 84.7), turned to 180 degrees
- moved R6 18.0 mm to (190.5, 79.6), turned to 180 degrees
- moved C4 17.8 mm to (198.1, 96.1)
- moved U1 17.8 mm to (203.2, 99.9)
- moved U2 11.7 mm to (195.6, 79.6), turned to 0 degrees
- moved C6 1.69 mm to (198.1, 68.2)
- moved C5 1.27 mm to (203.2, 83.4)
- moved U3 1.27 mm to (182.9, 69.5)
- renumbered C7 to C5, C8 to C6, J11 to J1, J6 to J10, J7 to J11, J4 to J12, J9 to J13, J10 to J2, J1 to J3, J2 to J4, J3 to J5, J12 to J6, J8 to J7, J13 to J8, J5 to J9, R6 to R1, R1 to R10, R2 to R11, R3 to R12, R16 to R13, R17 to R14, R18 to R15, R20 to R16, R21 to R17, R22 to R18, R4 to R19, R7 to R2, R5 to R20, R15 to R21, R19 to R22, R24 to R23, R23 to R24, R8 to R3, R9 to R4, R10 to R5, R11 to R6, R12 to R7, R13 to R8, R14 to R9, U3 to U2, U4 to U3
Connections:
- net +10V renamed 10V_REF
- net +10V_P renamed 10V_REF_P
- R10 pad 1: Net-(R1-Pad1) -> Net-(R10-Pad1)
- R11 pad 1: Net-(R1-Pad1) -> Net-(R10-Pad1)
- R12 pad 1: Net-(R1-Pad1) -> Net-(R10-Pad1)
- R13 pad 1: Net-(R16-Pad1) -> Net-(R13-Pad1)
- R13 pad 2: Net-(R12-Pad1) -> Net-(R13-Pad2)
- R14 pad 1: Net-(R17-Pad1) -> Net-(R14-Pad1)
- R14 pad 2: Net-(R13-Pad1) -> Net-(R14-Pad2)
- R16 pad 2: Net-(R16-Pad1) -> Net-(R13-Pad1)
- R17 pad 2: Net-(R17-Pad1) -> Net-(R14-Pad1)
- R19 pad 1: Net-(R24-Pad2) -> Net-(R19-Pad1)
- R19 pad 2: Net-(R1-Pad1) -> Net-(R10-Pad1)
- R20 pad 1: Net-(R15-Pad2) (its old number) -> Net-(R20-Pad1)
- R20 pad 2: Net-(R24-Pad2) -> Net-(R19-Pad1)
- R21 pad 1: Net-(R15-Pad1) (its old number) -> Net-(R21-Pad1)
- R21 pad 2: Net-(R15-Pad2) (its old number) -> Net-(R20-Pad1)
- R22 pad 2: Net-(R15-Pad1) (its old number) -> Net-(R21-Pad1)
- R23 pad 2: Net-(R24-Pad2) -> Net-(R19-Pad1)
- R7 pad 1: Net-(R12-Pad1) -> Net-(R13-Pad2)
- R8 pad 1: Net-(R13-Pad1) -> Net-(R14-Pad2)
- RV1 pad 1: INV1_P -> GND1
- RV1 pad 3: GND1 -> INV1_P
- RV2 pad 1: INV2_P -> GND1
- RV2 pad 3: GND1 -> INV2_P
- RV3 pad 1: INV3_P -> GND1
- RV3 pad 3: GND1 -> INV3_P
- U1 pad 1: Net-(R16-Pad1) -> Net-(R19-Pad1)
- U1 pad 2: Net-(R12-Pad1) -> Net-(R10-Pad1)
- U1 pad 3: NONINV1 -> GND
- U1 pad 5: NONINV2 -> NONINV1
- U1 pad 6: Net-(R13-Pad1) -> Net-(R13-Pad2)
- U1 pad 7: Net-(R17-Pad1) -> Net-(R13-Pad1)
- U1 pad 8: -12V -> Net-(R14-Pad1)
- U2 pad 4: +12V -> -12V
- U2 pad 7: -12V -> +12V
Routing:
- net NONINV1_P: track 122.2 -> 36.3 mm
- net NONINV2_P: track 115.1 -> 36.6 mm
- net NONINV3_P: track 115.7 -> 38.2 mm
- net Net-(R19-Pad1): track 0.00 -> 41.9 mm
- net Net-(R24-Pad2): track 35.1 -> 0.00 mm
- net Net-(R1-Pad1): track 28.0 -> 0.00 mm
- net Net-(R10-Pad1): track 0.00 -> 27.5 mm
- net Net-(R13-Pad2): track 0.00 -> 25.4 mm
- net NONINV3: track 87.1 -> 110.7 mm
- net Net-(R14-Pad2): track 0.00 -> 23.3 mm
- net +12V: track 87.2 -> 65.7 mm
- net Net-(R21-Pad1): track 0.00 -> 21.3 mm
- net Net-(R15-Pad1) (its old number): track 20.8 -> 0.00 mm
- net INV3: track 85.0 -> 105.0 mm
- net Net-(R12-Pad1): track 18.4 -> 0.00 mm
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
Commit message: Test points
Parts:
- added TP1: GND, ao_tht:TestPoint_THTPad_1.5x1.5mm_Drill0.7mm, B.Cu at (221.0, 44.0)
- added TP2: +12V, ao_tht:TestPoint_THTPad_D1.5mm_Drill0.7mm, B.Cu at (221.0, 47.9)
- added TP3: -12V, ao_tht:TestPoint_THTPad_D1.5mm_Drill0.7mm, B.Cu at (221.0, 51.7)
- added TP4: GND, ao_tht:TestPoint_THTPad_1.5x1.5mm_Drill0.7mm, F.Cu at (132.1, 112.6)
Routing:
- net -12V: track 69.5 -> 90.0 mm
- net +12V: track 65.7 -> 84.5 mm

Commit message: Better .gitignore; KiCad 6 version
Parts:
- added B1: Board, ao_tht:Board_Marker, F.Cu at (199.5, 42.0)
- added B2: Board, ao_tht:Board_Marker, F.Cu at (98.5, 20.0)
Connections:
- net OUT~SUM~ renamed OUT~{SUM}
- net OUT~SUM~_P renamed OUT~{SUM}_P
- U2 pad 1: Net-(U2-Pad1) -> unconnected-(U2-Pad1)
- U2 pad 5: Net-(U2-Pad5) -> unconnected-(U2-Pad5)
- U2 pad 8: Net-(U2-Pad8) -> unconnected-(U2-Pad8)
Other:
- outline, holes or cut-outs redrawn
- net class Default removed
- net class Power removed
- board text added: "+10V"
- board text added: "10"
- board text added: "Center"
- board text added: "G"
- board text added: "I1"
- board text added: "I2"
- board text added: "I3"
- board text added: "Jack"
- board text added: "N1"
- board text added: "N2"
- board text added: "N3"
- board text added: "O1"
- board text added: "O2"
- board text added: "O3"
- board text added: "Rich Holmes Jan 2022 CC0 1.0"
- board text added: "S"
- board text added: "S1"
- board text added: "S2"
- board text added: "S3"
- board text added: "~{S}"
- board text removed: "Rich Holmes Oct 2021 CC0 1.0"

Commit message: Catch up to 1st fab run version
Parts:
- removed J8: 3_pin_Molex_connector, ao_tht:Molex_KK-254_AE-6410-03A_1x03_P2.54mm_Vertical
- removed SW1: SW_SPDT, ao_tht:SPDT-toggle-switch-1M-series
Routing:
- net Net-(J8-Pad3): track 12.9 -> 0.00 mm
- net Net-(J8-Pad1): track 12.7 -> 0.00 mm
- net Net-(J8-Pad2): track 12.0 -> 0.00 mm
- net INV2_P: track 114.1 -> 113.1 mm
- net OUT2_P: track 33.5 -> 32.9 mm
Other:
- outline, holes or cut-outs redrawn

Commit message: Slot version of jacks
Parts:
- J10, J11, J12, J13, J3, J4, J5, J9: footprint ao_tht:Jack_6.35mm_PJ_629HAN -> ao_tht:Jack_6.35mm_PJ_629HAN_slots
- RV1, RV2, RV3: value 100k -> B100k
