File: Hardware/PCB/attenuverters/attenuverters.kicad_sch (KiCad schematic)
At the start: 64 parts, among them J1 Conn_01x16, J10 AudioJack2_SwitchT, J11 AudioJack2_SwitchT, J12 AudioJack2, J13 AudioJack2, J2 Conn_01x16, J3 AudioJack2, J4 AudioJack2, J5 AudioJack2, J6 3_pin_Molex_header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

Commit message: Catch up to 1st fab run version
Parts:
- B1, B2, GRAF1, GRAF2, H1, H2, H3, H4: now left out of the parts list
- RV1, RV2, RV3: value 100k -> (none)
- TP1: value GND -> (none); footprint ao_tht:TestPoint_THTPad_1.5x1.5mm_Drill0.7mm -> (none); Config (none) -> DNF; now left out of the parts list
- TP2, TP3: Config (none) -> DNF; now left out of the parts list
- TP4: value GND -> (none); footprint ao_tht:TestPoint_THTPad_1.5x1.5mm_Drill0.7mm -> (none); now left out of the parts list
Changed lines of the file:
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@@
     (stroke (width 0) (type default) (color 0 0 0 0))
   )
+  (polyline (pts (xy 91.44 130.81) (xy 138.43 130.81))
+    (stroke (width 0) (type default) (color 0 0 0 0))
+  )
   (wire (pts (xy 165.1 41.91) (xy 165.1 45.72))
     (stroke (width 0) (type default) (color 0 0 0 0))
@@
     (stroke (width 0) (type default) (color 0 0 0 0))
   )
+  (polyline (pts (xy 138.43 82.55) (xy 91.44 82.55))
+    (stroke (width 0) (type default) (color 0 0 0 0))
+  )
   (wire (pts (xy 66.04 48.26) (xy 63.5 48.26))
     (stroke (width 0) (type default) (color 0 0 0 0))
@@
     (stroke (width 0) (type default) (color 0 0 0 0))
   )
+  (polyline (pts (xy 91.44 82.55) (xy 91.44 130.81))
+    (stroke (width 0) (type default) (color 0 0 0 0))
+  )
   (wire (pts (xy 176.53 67.31) (xy 182.88 67.31))
     (stroke (width 0) (type default) (color 0 0 0 0))
@@
     (stroke (width 0) (type default) (color 0 0 0 0))
   )
-  (polyline (pts (xy 138.43 82.55) (xy 138.43 171.45))
+  (polyline (pts (xy 138.43 130.81) (xy 138.43 171.45))
     (stroke (width 0) (type default) (color 0 0 0 0))
   )
@@
   )
   (symbol (lib_id "ao_symbols:SW_SPDT") (at 227.33 101.6 0) (unit 1)
-    (in_bom yes) (on_board yes)
+    (in_bom yes) (on_board no)
     (property "Reference" "SW1" (id 0) (at 227.33 94.361 0))
     (property "Value" "SW_SPDT" (id 1) (at 227.33 96.6724 0))
@@
       (effects (font (size 1.27 1.27)) (justify right))
     )
-    (property "Value" "100k" (id 1) (at 174.7774 116.713 0)
+    (property "Value" "" (id 1) (at 174.7774 116.713 0)
       (effects (font (size 1.27 1.27)) (justify right))
     )
@@
       (effects (font (size 1.27 1.27)) hide)
     )
+    (pin "1")
+    (pin "2")
+    (pin "3")
     (pin "5")
     (pin "6")
     (pin "7")
+    (pin "10")
+    (pin "8")
+    (pin "9")
+    (pin "12")
+    (pin "13")
+    (pin "14")
+    (pin "11")
+    (pin "4")
   )
   (symbol (lib_id "ao_symbols:R") (at 55.88 34.29 270) (unit 1)
@@
   )
   (symbol (lib_id "ao_symbols:Graphic") (at 24.13 196.85 0) (unit 1)
-    (in_bom yes) (on_board yes)
+    (in_bom no) (on_board yes)
     (property "Reference" "GRAF1" (id 0) (at 31.1912 195.6816 0)
       (effects (font (size 1.27 1.27)) (justify left))
@@
       (effects (font (size 1.27 1.27)) (justify right))
     )
-    (property "Value" "100k" (id 1) (at 174.7774 139.573 0)
+    (property "Value" "" (id 1) (at 174.7774 139.573 0)
       (effects (font (size 1.27 1.27)) (justify right))
     )
@@
       (effects (font (size 1.27 1.27)) hide)
     )
+    (pin "1")
+    (pin "2")
+    (pin "3")
+    (pin "5")
+    (pin "6")
+    (pin "7")
     (pin "10")
     (pin "8")
     (pin "9")
+    (pin "12")
+    (pin "13")
+    (pin "14")
+    (pin "11")
+    (pin "4")
   )
   (symbol (lib_id "ao_symbols:R") (at 55.88 72.39 270) (unit 1)
@@
       (effects (font (size 1.27 1.27)) (justify right))
     )
-    (property "Value" "100k" (id 1) (at 174.7774 159.893 0)
+    (property "Value" "" (id 1) (at 174.7774 159.893 0)
       (effects (font (size 1.27 1.27)) (justify right))
     )
@@
     (pin "2")
     (pin "3")
+    (pin "5")
+    (pin "6")
+    (pin "7")
+    (pin "10")
+    (pin "8")
+    (pin "9")
+    (pin "12")
+    (pin "13")
+    (pin "14")
+    (pin "11")
+    (pin "4")
   )
   (symbol (lib_id "power:GND") (at 60.96 171.45 0) (unit 1)
@@
       (effects (font (size 1.27 1.27)) hide)
     )
+    (pin "1")
+    (pin "2")
+    (pin "3")
+    (pin "5")
+    (pin "6")
+    (pin "7")
+    (pin "10")
+    (pin "8")
+    (pin "9")
     (pin "12")
     (pin "13")
     (pin "14")
+    (pin "11")
+    (pin "4")
   )
   (symbol (lib_id "power:GND") (at 93.98 173.99 0) (unit 1)
@@
       (effects (font (size 1.27 1.27)) hide)
     )
+    (pin "1")
+    (pin "2")
+    (pin "3")
+    (pin "5")
+    (pin "6")
+    (pin "7")
+    (pin "10")
+    (pin "8")
+    (pin "9")
+    (pin "12")
+    (pin "13")
+    (pin "14")
     (pin "11")
     (pin "4")
@@
   )
   (symbol (lib_id "ao_symbols:TestPoint") (at 247.65 59.69 0) (unit 1)
-    (in_bom yes) (on_board yes)
+    (in_bom no) (on_board yes)
     (property "Reference" "TP1" (id 0) (at 249.1232 56.6928 0)
       (effects (font (size 1.27 1.27)) (justify left))
     )
-    (property "Value" "GND" (id 1) (at 249.1232 59.0042 0)
+    (property "Value" "" (id 1) (at 249.1232 59.0042 0)
       (effects (font (size 1.27 1.27)) (justify left))
     )
-    (property "Footprint" "ao_tht:TestPoint_THTPad_1.5x1.5mm_Drill0.7mm" (id 2) (at 252.73 59.69 0)
+    (property "Footprint" "" (id 2) (at 252.73 59.69 0)
       (effects (font (size 1.27 1.27)) hide)
     )
@@
       (effects (font (size 1.27 1.27)) hide)
     )
+    (property "Config" "DNF" (id 4) (at 247.65 59.69 0)
+      (effects (font (size 1.27 1.27)) hide)
+    )
     (pin "1")
   )
   (symbol (lib_id "ao_symbols:TestPoint") (at 247.65 67.31 0) (unit 1)
-    (in_bom yes) (on_board yes)
+    (in_bom no) (on_board yes)
     (property "Reference" "TP2" (id 0) (at 249.1232 64.3128 0)
       (effects (font (size 1.27 1.27)) (justify left))
@@
       (effects (font (size 1.27 1.27)) hide)
     )
+    (property "Config" "DNF" (id 4) (at 247.65 67.31 0)
+      (effects (font (size 1.27 1.27)) hide)
+    )
     (pin "1")
   )
   (symbol (lib_id "ao_symbols:TestPoint") (at 247.65 74.93 0) (unit 1)
-    (in_bom yes) (on_board yes)
+    (in_bom no) (on_board yes)
     (property "Reference" "TP3" (id 0) (at 249.1232 71.9328 0)
       (effects (font (size 1.27 1.27)) (justify left))
@@
       (effects (font (size 1.27 1.27)) hide)
     )
+    (property "Config" "DNF" (id 4) (at 247.65 74.93 0)
+      (effects (font (size 1.27 1.27)) hide)
+    )
     (pin "1")
   )
@@
   )
   (symbol (lib_id "Connector:TestPoint") (at 247.65 100.33 0) (unit 1)
-    (in_bom yes) (on_board yes)
+    (in_bom no) (on_board yes)
     (property "Reference" "TP4" (id 0) (at 249.1232 97.3328 0)
       (effects (font (size 1.27 1.27)) (justify left))
     )
-    (property "Value" "GND" (id 1) (at 249.1232 99.6442 0)
+    (property "Value" "" (id 1) (at 249.1232 99.6442 0)
       (effects (font (size 1.27 1.27)) (justify left))
     )
-    (property "Footprint" "ao_tht:TestPoint_THTPad_1.5x1.5mm_Drill0.7mm" (id 2) (at 252.73 100.33 0)
+    (property "Footprint" "" (id 2) (at 252.73 100.33 0)
       (effects (font (size 1.27 1.27)) hide)
     )
@@
   )
   (symbol (lib_id "ao_symbols:MountingHole") (at 45.72 196.85 0) (unit 1)
-    (in_bom yes) (on_board yes)
+    (in_bom no) (on_board yes)
     (property "Reference" "H1" (id 0) (at 48.26 195.6816 0)
       (effects (font (size 1.27 1.27)) (justify left))
@@
   )
   (symbol (lib_id "ao_symbols:MountingHole") (at 64.77 196.85 0) (unit 1)
-    (in_bom yes) (on_board yes)
+    (in_bom no) (on_board yes)
     (property "Reference" "H2" (id 0) (at 67.31 195.6816 0)
       (effects (font (size 1.27 1.27)) (justify left))
@@
   )
   (symbol (lib_id "ao_symbols:MountingHole") (at 245.11 153.67 0) (unit 1)
-    (in_bom yes) (on_board yes)
+    (in_bom no) (on_board yes)
     (property "Reference" "H3" (id 0) (at 247.65 152.5016 0)
       (effects (font (size 1.27 1.27)) (justify left))
@@
   )
   (symbol (lib_id "ao_symbols:MountingHole") (at 245.11 158.75 0) (unit 1)
-    (in_bom yes) (on_board yes)
+    (in_bom no) (on_board yes)
     (property "Reference" "H4" (id 0) (at 247.65 157.5816 0)
       (effects (font (size 1.27 1.27)) (justify left))
@@
   )
   (symbol (lib_id "ao_symbols:3_pin_Molex_connector") (at 213.36 101.6 0) (mirror y) (unit 1)
-    (in_bom yes) (on_board yes)
+    (in_bom yes) (on_board no)
     (property "Reference" "J8" (id 0) (at 215.4428 93.5482 0))
     (property "Value" "3_pin_Molex_connector" (id 1) (at 215.4428 95.8596 0))
@@
   )
   (symbol (lib_id "ao_symbols:Graphic") (at 248.92 147.32 0) (unit 1)
-    (in_bom yes) (on_board yes)
+    (in_bom no) (on_board yes)
     (property "Reference" "GRAF2" (id 0) (at 255.9812 146.1516 0)
       (effects (font (size 1.27 1.27)) (justify left))
@@
   )
   (symbol (lib_id "ao_symbols:Board") (at 252.73 90.17 0) (unit 1)
-    (in_bom yes) (on_board yes) (fields_autoplaced)
+    (in_bom no) (on_board yes) (fields_autoplaced)
     (property "Reference" "B2" (id 0) (at 258.445 89.2615 0)
       (effects (font (size 1.27 1.27)) (justify left))
@@
   )
   (symbol (lib_id "ao_symbols:Board") (at 91.44 198.12 0) (unit 1)
-    (in_bom yes) (on_board yes) (fields_autoplaced)
+    (in_bom no) (on_board yes) (fields_autoplaced)
     (property "Reference" "B1" (id 0) (at 97.155 197.2115 0)
       (effects (font (size 1.27 1.27)) (justify left))
@@
     )
     (path "/00000000-0000-0000-0000-00006167d75a"
-      (reference "RV1") (unit 1) (value "100k") (footprint "ao_tht:Potentiometer_Alpha_RA6020F_Single_Slide")
+      (reference "RV1") (unit 1) (value "B100k") (footprint "ao_tht:Potentiometer_Alpha_RA6020F_Single_Slide")
     )
     (path "/00000000-0000-0000-0000-0000616965cc"
-      (reference "RV2") (unit 1) (value "100k") (footprint "ao_tht:Potentiometer_Alpha_RA6020F_Single_Slide")
+      (reference "RV2") (unit 1) (value "B100k") (footprint "ao_tht:Potentiometer_Alpha_RA6020F_Single_Slide")
     )
     (path "/00000000-0000-0000-0000-00006169cde5"
-      (reference "RV3") (unit 1) (value "100k") (footprint "ao_tht:Potentiometer_Alpha_RA6020F_Single_Slide")
+      (reference "RV3") (unit 1) (value "B100k") (footprint "ao_tht:Potentiometer_Alpha_RA6020F_Single_Slide")
     )
     (path "/00000000-0000-0000-0000-00006167bdd2"

Commit message: Slot version of jacks
Parts:
- J10, J11, J12, J13, J3, J4, J5, J9: footprint ao_tht:Jack_6.35mm_PJ_629HAN -> (none)
- RV1, RV2, RV3: value (none) -> B100k
- TP1, TP4: value (none) -> GND; footprint (none) -> ao_tht:TestPoint_THTPad_1.5x1.5mm_Drill0.7mm
Changed lines of the file:
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@@
   (title_block
     (title "Attenuverters")
-    (date "2022-01-29")
+    (date "2022-03-26")
     (company "Rich Holmes / Analog Output")
     (comment 1 "or neighboring rights to this work. Published from United States.")
@@
       (effects (font (size 1.27 1.27)) (justify right))
     )
-    (property "Footprint" "ao_tht:Jack_6.35mm_PJ_629HAN" (id 2) (at 154.94 111.76 0)
+    (property "Footprint" "" (id 2) (at 154.94 111.76 0)
       (effects (font (size 1.27 1.27)) hide)
     )
@@
       (effects (font (size 1.27 1.27)) (justify right))
     )
-    (property "Value" "" (id 1) (at 174.7774 116.713 0)
+    (property "Value" "B100k" (id 1) (at 174.7774 116.713 0)
       (effects (font (size 1.27 1.27)) (justify right))
     )
@@
       (effects (font (size 1.27 1.27)) (justify right))
     )
-    (property "Footprint" "ao_tht:Jack_6.35mm_PJ_629HAN" (id 2) (at 214.63 118.11 0)
+    (property "Footprint" "" (id 2) (at 214.63 118.11 0)
       (effects (font (size 1.27 1.27)) hide)
     )
@@
       (effects (font (size 1.27 1.27)) (justify right))
     )
-    (property "Footprint" "ao_tht:Jack_6.35mm_PJ_629HAN" (id 2) (at 251.46 130.81 0)
+    (property "Footprint" "" (id 2) (at 251.46 130.81 0)
       (effects (font (size 1.27 1.27)) hide)
     )
@@
       (effects (font (size 1.27 1.27)) (justify right))
     )
-    (property "Footprint" "ao_tht:Jack_6.35mm_PJ_629HAN" (id 2) (at 154.94 132.08 0)
+    (property "Footprint" "" (id 2) (at 154.94 132.08 0)
       (effects (font (size 1.27 1.27)) hide)
     )
@@
       (effects (font (size 1.27 1.27)) (justify right))
     )
-    (property "Value" "" (id 1) (at 174.7774 139.573 0)
+    (property "Value" "B100k" (id 1) (at 174.7774 139.573 0)
       (effects (font (size 1.27 1.27)) (justify right))
     )
@@
       (effects (font (size 1.27 1.27)) (justify right))
     )
-    (property "Footprint" "ao_tht:Jack_6.35mm_PJ_629HAN" (id 2) (at 214.63 135.89 0)
+    (property "Footprint" "" (id 2) (at 214.63 135.89 0)
       (effects (font (size 1.27 1.27)) hide)
     )
@@
       (effects (font (size 1.27 1.27)) (justify right))
     )
-    (property "Footprint" "ao_tht:Jack_6.35mm_PJ_629HAN" (id 2) (at 154.94 152.4 0)
+    (property "Footprint" "" (id 2) (at 154.94 152.4 0)
       (effects (font (size 1.27 1.27)) hide)
     )
@@
       (effects (font (size 1.27 1.27)) (justify right))
     )
-    (property "Value" "" (id 1) (at 174.7774 159.893 0)
+    (property "Value" "B100k" (id 1) (at 174.7774 159.893 0)
       (effects (font (size 1.27 1.27)) (justify right))
     )
@@
       (effects (font (size 1.27 1.27)) (justify right))
     )
-    (property "Footprint" "ao_tht:Jack_6.35mm_PJ_629HAN" (id 2) (at 214.63 153.67 0)
+    (property "Footprint" "" (id 2) (at 214.63 153.67 0)
       (effects (font (size 1.27 1.27)) hide)
     )
@@
       (effects (font (size 1.27 1.27)) (justify right))
     )
-    (property "Footprint" "ao_tht:Jack_6.35mm_PJ_629HAN" (id 2) (at 251.46 115.57 0)
+    (property "Footprint" "" (id 2) (at 251.46 115.57 0)
       (effects (font (size 1.27 1.27)) hide)
     )
@@
       (effects (font (size 1.27 1.27)) (justify left))
     )
-    (property "Value" "" (id 1) (at 249.1232 59.0042 0)
+    (property "Value" "GND" (id 1) (at 249.1232 59.0042 0)
       (effects (font (size 1.27 1.27)) (justify left))
     )
-    (property "Footprint" "" (id 2) (at 252.73 59.69 0)
+    (property "Footprint" "ao_tht:TestPoint_THTPad_1.5x1.5mm_Drill0.7mm" (id 2) (at 252.73 59.69 0)
       (effects (font (size 1.27 1.27)) hide)
     )
@@
       (effects (font (size 1.27 1.27)) (justify left))
     )
-    (property "Value" "" (id 1) (at 249.1232 99.6442 0)
+    (property "Value" "GND" (id 1) (at 249.1232 99.6442 0)
       (effects (font (size 1.27 1.27)) (justify left))
     )
-    (property "Footprint" "" (id 2) (at 252.73 100.33 0)
+    (property "Footprint" "ao_tht:TestPoint_THTPad_1.5x1.5mm_Drill0.7mm" (id 2) (at 252.73 100.33 0)
       (effects (font (size 1.27 1.27)) hide)
     )
@@
     )
     (path "/00000000-0000-0000-0000-00006167ac41"
-      (reference "J3") (unit 1) (value "AudioJack2") (footprint "ao_tht:Jack_6.35mm_PJ_629HAN")
+      (reference "J3") (unit 1) (value "AudioJack2") (footprint "ao_tht:Jack_6.35mm_PJ_629HAN_slots")
     )
     (path "/00000000-0000-0000-0000-000061696597"
-      (reference "J4") (unit 1) (value "AudioJack2") (footprint "ao_tht:Jack_6.35mm_PJ_629HAN")
+      (reference "J4") (unit 1) (value "AudioJack2") (footprint "ao_tht:Jack_6.35mm_PJ_629HAN_slots")
     )
     (path "/00000000-0000-0000-0000-00006169cdb1"
-      (reference "J5") (unit 1) (value "AudioJack2") (footprint "ao_tht:Jack_6.35mm_PJ_629HAN")
+      (reference "J5") (unit 1) (value "AudioJack2") (footprint "ao_tht:Jack_6.35mm_PJ_629HAN_slots")
     )
     (path "/00000000-0000-0000-0000-000061cddffb"
@@
     )
     (path "/00000000-0000-0000-0000-000061688e07"
-      (reference "J9") (unit 1) (value "AudioJack2_SwitchT") (footprint "ao_tht:Jack_6.35mm_PJ_629HAN")
+      (reference "J9") (unit 1) (value "AudioJack2_SwitchT") (footprint "ao_tht:Jack_6.35mm_PJ_629HAN_slots")
     )
     (path "/00000000-0000-0000-0000-00006169661b"
-      (reference "J10") (unit 1) (value "AudioJack2_SwitchT") (footprint "ao_tht:Jack_6.35mm_PJ_629HAN")
+      (reference "J10") (unit 1) (value "AudioJack2_SwitchT") (footprint "ao_tht:Jack_6.35mm_PJ_629HAN_slots")
     )
     (path "/00000000-0000-0000-0000-00006169ce34"
-      (reference "J11") (unit 1) (value "AudioJack2_SwitchT") (footprint "ao_tht:Jack_6.35mm_PJ_629HAN")
+      (reference "J11") (unit 1) (value "AudioJack2_SwitchT") (footprint "ao_tht:Jack_6.35mm_PJ_629HAN_slots")
     )
     (path "/00000000-0000-0000-0000-000061720573"
-      (reference "J12") (unit 1) (value "AudioJack2") (footprint "ao_tht:Jack_6.35mm_PJ_629HAN")
+      (reference "J12") (unit 1) (value "AudioJack2") (footprint "ao_tht:Jack_6.35mm_PJ_629HAN_slots")
     )
     (path "/00000000-0000-0000-0000-00006168bca1"
-      (reference "J13") (unit 1) (value "AudioJack2") (footprint "ao_tht:Jack_6.35mm_PJ_629HAN")
+      (reference "J13") (unit 1) (value "AudioJack2") (footprint "ao_tht:Jack_6.35mm_PJ_629HAN_slots")
     )
     (path "/00000000-0000-0000-0000-00006167e358"
