File: Hardware/Panel/attenuverters_panel/attenuverters_panel.kicad_pcb (KiCad board)
At the start: 2 copper layers, 75 x 200 mm, 17 parts

Commit message: Rear panel labels
Other:
- board text added: "10V/jack switch"
- board text added: "In 1 jack"
- board text added: "In 1 slider"
- board text added: "In 2 jack"
- board text added: "In 2 slider"
- board text added: "In 3 jack"
- board text added: "In 3 slider"
- board text added: "Out 1 jack"
- board text added: "Out 2 jack"
- board text added: "Out 3 jack"
- board text added: "Sum out jack"
- board text added: "~Sum~ out jack"

Commit message: Better .gitignore; KiCad 6 version
Other:
- net class Default removed
- board text added: "10V terminal"
- board text added: "Jack terminal"
- board text added: "Panel design by Rich Holmes CC0 1.0 Jan 2022 JLCJLCJLCJLC"
- board text added: "~{Sum} out jack"
- board text removed: "Panel design by Rich Holmes CC0 1.0 Oct 2021 JLCJLCJLCJLC"
- board text removed: "~Sum~ out jack"

Commit message: Catch up to 1st fab run version
Changed lines of the file:
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@@
     (effects (font (size 1 1) (thickness 0.15)) (justify mirror))
   )
-  (zone (net 1) (net_name "GND") (layer "F.Cu") (hatch edge 0.508)
+  (zone (net 1) (net_name "GND") (layers F&B.Cu) (hatch edge 0.508)
     (connect_pads (clearance 0.508))
-    (min_thickness 0.254)
+    (min_thickness 0.254) (filled_areas_thickness no)
     (fill yes (thermal_gap 0.508) (thermal_bridge_width 0.508))
     (polygon
       (pts
-        (xy 96.1 212.6)
-        (xy 11.1 212.6)
-        (xy 11.1 2.6)
-        (xy 96.1 2.6)
+        (xy 91.1 207.6)
+        (xy 16.1 207.6)
+        (xy 16.1 7.6)
+        (xy 91.1 7.6)
       )
     )
-  )
-  (zone (net 1) (net_name "GND") (layer "B.Cu") (hatch edge 0.508)
-    (connect_pads (clearance 0.508))
-    (min_thickness 0.254)
-    (fill yes (thermal_gap 0.508) (thermal_bridge_width 0.508))
-    (polygon
-      (pts
-        (xy 96.1 212.6)
-        (xy 11.1 212.6)
-        (xy 11.1 2.6)
-        (xy 96.1 2.6)
-      )
-    )
